Commit message: rename wheel in communication protocol

File: src/omni_gazebo/urdf/omni_base.urdf (robot description, URDF)
Before this commit: robot sirius, 4 links, 3 joints
Links:
- removed link front_wheel
- removed link left_wheel
- removed link right_wheel
- added link wheel_A, mass 10; collision cylinder length=0.04 radius=0.06; visual cylinder length=0.04 radius=0.06
- added link wheel_B, mass 10; collision cylinder length=0.03 radius=0.08; visual cylinder length=0.04 radius=0.06
- added link wheel_C, mass 10; collision cylinder length=0.04 radius=0.06; visual cylinder length=0.04 radius=0.06
Joints:
- removed joint base_to_front_wheel
- removed joint base_to_left_wheel
- removed joint base_to_right_wheel
- added joint base_to_wheel_A: type fixed, parent base_link, child wheel_A, origin xyz=0.124525 -0.21568 -0.08 rpy=0 0 0
- added joint base_to_wheel_B: type fixed, parent base_link, child wheel_B, origin xyz=0.124525 0.21568 -0.08 rpy=0 0 0
- added joint base_to_wheel_C: type fixed, parent base_link, child wheel_C, origin xyz=-0.24905 0 -0.08 rpy=0 0 0

Commit message: Revert "rename wheel in communication protocol"
This reverts commit 36ba005b4de9f34fd72cb6af41d1b1e33149ec96.

File: src/omni_gazebo/urdf/omni_base.urdf (robot description, URDF)
Before this commit: robot sirius, 4 links, 3 joints
Links:
- removed link wheel_A
- removed link wheel_B
- removed link wheel_C
- added link front_wheel, mass 10; collision cylinder length=0.04 radius=0.06; visual cylinder length=0.04 radius=0.06
- added link left_wheel, mass 10; collision cylinder length=0.04 radius=0.06; visual cylinder length=0.04 radius=0.06
- added link right_wheel, mass 10; collision cylinder length=0.03 radius=0.08; visual cylinder length=0.04 radius=0.06
Joints:
- removed joint base_to_wheel_A
- removed joint base_to_wheel_B
- removed joint base_to_wheel_C
- added joint base_to_front_wheel: type fixed, parent base_link, child front_wheel, origin xyz=0.24905 0 -0.08 rpy=0 0 0
- added joint base_to_left_wheel: type fixed, parent base_link, child left_wheel, origin xyz=-0.124525 0.21568 -0.08 rpy=0 0 0
- added joint base_to_right_wheel: type fixed, parent base_link, child right_wheel, origin xyz=-0.124525 -0.21568 -0.08 rpy=0 0 0

Commit message: rename wheel in communication protocol

File: src/omni_gazebo/urdf/omni_base.urdf (robot description, URDF)
Before this commit: robot sirius, 4 links, 3 joints
Links:
- removed link front_wheel
- removed link left_wheel
- removed link right_wheel
- added link wheel_A, mass 10; collision cylinder length=0.03 radius=0.08; visual cylinder length=0.04 radius=0.06
- added link wheel_B, mass 10; collision cylinder length=0.04 radius=0.06; visual cylinder length=0.04 radius=0.06
- added link wheel_C, mass 10; collision cylinder length=0.04 radius=0.06; visual cylinder length=0.04 radius=0.06
Joints:
- removed joint base_to_front_wheel
- removed joint base_to_left_wheel
- removed joint base_to_right_wheel
- added joint base_to_wheel_A: type fixed, parent base_link, child wheel_A, origin xyz=0.124525 0.21568 -0.08 rpy=0 0 0
- added joint base_to_wheel_B: type fixed, parent base_link, child wheel_B, origin xyz=0.124525 -0.21568 -0.08 rpy=0 0 0
- added joint base_to_wheel_C: type fixed, parent base_link, child wheel_C, origin xyz=0.24905 0 -0.08 rpy=0 0 0

Commit message: fix wheel_C origin

File: src/omni_gazebo/urdf/omni_base.urdf (robot description, URDF)
Before this commit: robot sirius, 4 links, 3 joints
Joints:
- joint base_to_wheel_C: origin xyz=0.24905 0 -0.08 rpy=0 0 0 -> xyz=-0.24905 0 -0.08 rpy=0 0 0
